Commit message: final task, first part

File: src/brita_r2d2/urdf/r2d2.urdf (robot description, URDF)
Before this commit: robot macroed, 6 links, 5 joints
Links:
- added link base_scan, mass 0.114; collision cylinder length=0.0315 radius=0.055; visual mesh filename=package://turtlebot3_description/meshes/sensors/lds.stl scale=0.001 0.001 0.001
Joints:
- added joint scan_joint: type fixed, parent box, child base_scan, origin xyz=0 0 0.06 rpy=0 0 0

File: src/brita_r2d2/urdf/r2d2.urdf.xacro (robot description, xacro)
@@ -237,5 +237,5 @@
     <xacro:default_inertial mass="1"/>
   </link>
-    <joint name="lens_tobox" type="revolute">
+  <joint name="lens_tobox" type="revolute">
     <parent link="box"/>
     <child link="lens"/>
@@ -244,3 +244,62 @@
     <axis xyz="0 8 0"/>
   </joint>
+  <link name="base_scan">
+    <visual>
+      <origin xyz="-0.01 0 0.02" rpy="0 0 0"/>
+      <geometry>
+        <mesh filename="package://turtlebot3_description/meshes/sensors/lds.stl" scale="0.001 0.001 0.001"/>
+      </geometry>
+      <material name="black"/>
+    </visual>
+    <collision>
+      <origin xyz="0.015 0 0.1" rpy="0 0 0"/>
+      <geometry>
+        <cylinder length="0.0315" radius="0.055"/>
+      </geometry>
+    </collision>
+    <inertial>
+      <mass value="0.114" />
+      <origin xyz="0 0 0" />
+      <inertia ixx="0.001" ixy="0.0" ixz="0.0"
+               iyy="0.001" iyz="0.0"
+               izz="0.001" />
+    </inertial>
+  </link>
+  <joint name="scan_joint" type="fixed">
+    <parent link="box"/>
+    <child link="base_scan"/>
+    <origin xyz="0 0 0.06" rpy="0 0 0"/>
+  </joint>
+  <gazebo reference="base_scan">
+    <material>Gazebo/FlatBlack</material>
+     <sensor type="ray" name="lds_lfcd_sensor">
+      <pose>0 0 0 0 0 0</pose>
+       <visualize>false</visualize>
+        <update_rate>5</update_rate>
+         <ray>
+          <scan>
+           <horizontal>
+            <samples>360</samples>
+            <resolution>1</resolution>
+            <min_angle>0.0</min_angle>
+            <max_angle>6.28319</max_angle>
+           </horizontal>
+          </scan>
+          <range>
+           <min>0.120</min>
+           <max>3.5</max>
+           <resolution>0.015</resolution>
+          </range>
+          <noise>
+           <type>gaussian</type>
+           <mean>0.0</mean>
+           <stddev>0.01</stddev>
+          </noise>
+         </ray>
+         <plugin name="gazebo_ros_lds_lfcd_controller" filename="libgazebo_ros_laser.so">
+          <topicName>scan</topicName>
+          <frameName>base_scan</frameName>
+         </plugin>
+      </sensor>
+  </gazebo>
 </robot>
